File: _autosave-ice4pi.kicad_pcb (KiCad board)
At the start: 4 copper layers, 85 x 56 mm, 32 parts, among them J1 Conn_02x03, J2 Raspberry_Pi_2_3, J3 USB_C_Receptacle_USB2.0, J5 RJ45_Abracon_ARJP11A-MASA-B-A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, U1 ENC28J60x-SS, U2 DSC1001DE1-025.0000

Commit message: feat: commit 2
Parts:
- added R3: 50, Resistor_SMD:R_0402_1005Metric, F.Cu at (119.5, 78.5)
- moved C10 0.48 mm to (119.5, 77.5)
Routing:
- net Net-(J5-RCT): track 18.6 -> 23.3 mm, vias 0 -> 2
- net GND: track 14.6 -> 13.2 mm, vias 10 -> 9
- net /TPIN+: track 35.6 -> 34.4 mm
